Commit message: [Task 3.111] Fixed all teleop issues with python file [CMakeLists.txt] Removed unnecessary lines [config/config_controllers.yaml] Tuned PID values [src/teleop_template.py] Fixed errors in teleop [urdf/rocr.urdf] Changed joint types [urdf/rocr_integration.urdf.xacro] Fixed error with plugin

File: urdf/rocr.urdf (robot description, URDF)
Before this commit: robot rocr, 17 links, 16 joints
Joints:
- joint joint_front_left_axle: limit lower=0 upper=0 effort=0 velocity=0 -> lower=-.35 upper=0.35 effort=1 velocity=0; type revolute -> continuous
- joint joint_front_right_axle: limit lower=0 upper=0 effort=0 velocity=0 -> lower=-0.35 upper=0.35 effort=1 velocity=0; type revolute -> continuous
- joint joint_rear_axle: limit lower=-1000000 upper=20 effort=10 velocity=100 -> (none); type revolute -> continuous

File: urdf/rocr_integration.urdf.xacro (robot description, xacro)
@@ -48,4 +48,6 @@
 		<plugin name="gazebo_ros_control" filename="libgazebo_ros_control.so">
 			<robotNamespace>/rocr</robotNamespace>
+			<robotSimType>gazebo_ros_control/DefaultRobotHWSim</robotSimType>
+			<legacyModeNS>true</legacyModeNS>
 		</plugin>
 	</gazebo>
