Commit message: [Task 3.08] Generated new output file to check if lidar and rocr is interagted properly

File: output.urdf (robot description, URDF)
Before this commit: robot rocr, 19 links, 18 joints
Joints:
- joint joint_front_left_axle: limit lower=-0.35 upper=0.35 effort=10 velocity=0 -> lower=-.35 upper=0.35 effort=1 velocity=0; type revolute -> continuous
- joint joint_front_right_axle: limit lower=-0.35 upper=0.35 effort=10 velocity=0 -> lower=-0.35 upper=0.35 effort=1 velocity=0; type revolute -> continuous
- joint joint_rear_axle: limit lower=-1000000 upper=20 effort=10 velocity=100 -> (none); type revolute -> continuous
