Commit message: [Task 4.01] Fixed the error with lidar not spawning

File: rocr/urdf/ydlidar.urdf (robot description, URDF)
Before this commit: robot ydlidar, 2 links, 1 joints
Links:
- link base_laser: geometry collision mesh filename=package://rocr/meshes/ydlidar.dae; visual mesh filename=package://rocr/meshes/ydlidar.dae
