Commit message: [Task 4.07] Added objects to pick up

File: rocr/urdf/rocr_integration.urdf.xacro (robot description, xacro)
@@ -7,4 +7,5 @@
 	<xacro:include filename="$(find rocr)/urdf/rocr.urdf" />
 	<xacro:include filename="$(find rocr)/urdf/ydlidar.urdf" />
+	<!-- <xacro:include filename="$(find rocr)/urdf/object.urdf" /> -->
 <!-- Add your gazebo sensors here -->
 <gazebo reference="base_laser">
@@ -64,3 +65,14 @@
       link="base_laser" />
   </joint>
+  <!-- <joint
+  name="object 1"
+  type="floating">
+  <origin
+	xyz="-1.25 -0.05 0.028"
+	rpy="0 0 3.14" />
+  <parent
+	link="base_link" />
+  <child
+	link="object" />
+  </joint> -->
 </robot>
