Commit message: [Task 4.03] Working on adding controllers for arms

File: rocr/urdf/rocr.urdf (robot description, URDF)
Before this commit: robot rocr, 17 links, 16 joints
Links:
- link link_pinion: geometry visual mesh filename=package://rocr/meshes/link_pinion.STL
Joints:
- joint joint_left_arm: limit lower=0 upper=0 effort=0 velocity=0 -> lower=-0.2 upper=0.2 effort=1000 velocity=0.5; type prismatic -> fixed
- joint joint_right_arm: limit lower=0 upper=0 effort=0 velocity=0 -> lower=-0.2 upper=0.2 effort=1000 velocity=0.5

Commit message: [Task 4.06] Fixed all known issues with teleop

File: rocr/urdf/rocr.urdf (robot description, URDF)
Before this commit: robot rocr, 17 links, 16 joints
Links:
- removed link link_bolt
- removed link link_pinion
- link link_front_left_axle: mass 0.00966461047960184 -> 0.00980151610171137
- link link_front_left_rim: mass 0.0118944183288657 -> 0.0269891429421557
- link link_front_left_tyre: mass 0.000894793246519236 -> 0.00176187281891002
- link link_front_right_axle: mass 0.00966461047960182 -> 0.00980150843161576
- link link_front_right_rim: mass 0.0118944183288657 -> 0.0269891429421557
- link link_front_right_tyre: mass 0.000894793246519238 -> 0.00176187281891002
- link link_left_arm: mass 1.1924981757879 -> 0.160992890586137
- link link_rear_axle: mass 0.0146411571669772 -> 0.0152217234982576
- link link_rear_left_rim: mass 0.0118944183288657 -> 0.0269891429421556
- link link_rear_left_tyre: mass 0.000894793246519235 -> 0.00176187281891002
- link link_rear_right_rim: mass 0.0118944183288657 -> 0.0269891429421557
- link link_rear_right_tyre: mass 0.000894793246519237 -> 0.00176187281891002
- link link_right_arm: mass 1.22458311377959 -> 0.165316765586137
Joints:
- removed joint joint_bolt
- removed joint joint_pinion
- joint joint_front_left_axle: limit lower=-.35 upper=0.35 effort=1 velocity=0 -> lower=0 upper=0.0 effort=1 velocity=0; origin xyz=-0.16 -0.074 -0.0346 rpy=-1.5708 0 -1.5708 -> xyz=-0.16 -0.074 -0.0346 rpy=1.5708 0 -1.6484
- joint joint_front_left_rim: origin xyz=0.009 0.027 0 rpy=-1.5708 -0.51596 1.5708 -> xyz=0.0030721 -0.027 0 rpy=-1.5708 1.1039 1.5708
- joint joint_front_left_tyre: origin xyz=0 0 -0.006 rpy=0 0 0.53015 -> xyz=0 0 0 rpy=3.1416 0 -0.81007
- joint joint_front_right_axle: limit lower=-0.35 upper=0.35 effort=1 velocity=0 -> lower=0 upper=0 effort=1 velocity=0
- joint joint_front_right_rim: origin xyz=0.009 -0.027 0 rpy=1.5708 0.2483 -1.5708 -> xyz=0.003 -0.027 0 rpy=1.5708 -0.93241 -1.5708
- joint joint_front_right_tyre: origin xyz=0 0 -0.006 rpy=0 0 1.197 -> xyz=0 0 -0.012 rpy=0 0 0.63839
- joint joint_left_arm: axis 0 0 0 -> 0 0 1; limit lower=-0.2 upper=0.2 effort=1000 velocity=0.5 -> lower=-1.5 upper=3.5 effort=1 velocity=0.2; origin xyz=-0.214 -0.11955 -0.074 rpy=1.5708 0 0 -> xyz=-0.214 0.066422 -0.072 rpy=1.5708 0 0; type fixed -> prismatic
- joint joint_rear_axle: origin xyz=-0.04 0 -0.0616 rpy=1.5707963267949 0.707024824141767 0 -> xyz=-0.04 0 -0.0616 rpy=1.5708 0 0
- joint joint_rear_left_rim: origin xyz=0 0 0.089 rpy=3.14159265358979 0 -0.351698544940136 -> xyz=0 0 0.089 rpy=3.1416 0 -2.7485
- joint joint_rear_left_tyre: origin xyz=0 0 0.00600000000000001 rpy=3.14159265358979 0 3.14159265358979 -> xyz=0 0 0.012 rpy=3.14159265358979 0 -2.74849784316327
- joint joint_rear_right_rim: origin xyz=0 0 0 rpy=0 0 0.24991380443404 -> xyz=0 0 0 rpy=0 0 0
- joint joint_rear_right_tyre: origin xyz=0 0 0 rpy=0 0 2.8695961764224 -> xyz=0 0 0 rpy=0 0 0
- joint joint_right_arm: axis 0 0 0 -> 0 0 1; limit lower=-0.2 upper=0.2 effort=1000 velocity=0.5 -> lower=-1.5 upper=3.5 effort=1 velocity=0.2; origin xyz=-0.36753 0.030166 -0.074 rpy=1.5708 0 0 -> xyz=-0.36753 0 -0.072 rpy=1.5708 0 0

Commit message: [Task 4.09] Fixed model issues

File: rocr/urdf/rocr.urdf (robot description, URDF)
Before this commit: robot rocr, 15 links, 14 joints
Links:
- removed link link_front_left_axle
- removed link link_front_left_rim
- removed link link_front_left_tyre
- removed link link_front_right_axle
- removed link link_front_right_rim
- removed link link_front_right_tyre
- removed link link_rear_axle
- removed link link_rear_left_rim
- removed link link_rear_left_tyre
- removed link link_rear_right_rim
- removed link link_rear_right_tyre
- added link link_left_rim, mass 0.400654705302582; collision mesh filename=package://rocr/meshes/link_left_rim.STL; visual mesh filename=package://rocr/meshes/link_left_rim.STL
- added link link_left_tyre, mass 0.00856487122656644; collision mesh filename=package://rocr/meshes/link_left_tyre.STL; visual mesh filename=package://rocr/meshes/link_left_tyre.STL
- added link link_rear_wheel, mass 0.0168994178831651; collision mesh filename=package://rocr/meshes/link_rear_wheel.STL; visual mesh filename=package://rocr/meshes/link_rear_wheel.STL
- added link link_right_rim, mass 0.400654705302582; collision mesh filename=package://rocr/meshes/link_right_rim.STL; visual mesh filename=package://rocr/meshes/link_right_rim.STL
- added link link_right_tyre, mass 0.00856487122656644; collision mesh filename=package://rocr/meshes/link_right_tyre.STL; visual mesh filename=package://rocr/meshes/link_right_tyre.STL
- link base_link: mass 10.6823173170711 -> 8.3349118107069
Joints:
- removed joint joint_front_left_axle
- removed joint joint_front_left_rim
- removed joint joint_front_left_tyre
- removed joint joint_front_right_axle
- removed joint joint_front_right_rim
- removed joint joint_front_right_tyre
- removed joint joint_rear_axle
- removed joint joint_rear_left_rim
- removed joint joint_rear_left_tyre
- removed joint joint_rear_right_rim
- removed joint joint_rear_right_tyre
- added joint joint_left_rim: type continuous, parent base_link, child link_left_rim, origin xyz=-0.175 -0.092 -0.041947 rpy=1.5708 -0.002359 3.1416, axis 0 0 1
- added joint joint_left_tyre: type fixed, parent link_left_rim, child link_left_tyre, origin xyz=0 0 0 rpy=3.1416 0 3.1392, axis 0 0 0
- added joint joint_rear_wheel: type continuous, parent base_link, child link_rear_wheel, origin xyz=-0.035562 -0.0445 -0.01849 rpy=1.5708 0 0, axis 0 1 0
- added joint joint_right_rim: type continuous, parent base_link, child link_right_rim, origin xyz=-0.175 0.003 -0.041947 rpy=1.5708 -0.40272 0, axis 0 0 1
- added joint joint_right_tyre: type fixed, parent link_right_rim, child link_right_tyre, origin xyz=0 0 -0.022 rpy=0 0 -0.40272, axis 0 0 0
- joint joint_left_arm: limit lower=-1.5 upper=3.5 effort=1 velocity=0.2 -> lower=0 upper=0 effort=0 velocity=0; origin xyz=-0.214 0.066422 -0.072 rpy=1.5708 0 0 -> xyz=-0.214 0.066815 -0.072 rpy=1.5708 0 0
- joint joint_right_arm: limit lower=-1.5 upper=3.5 effort=1 velocity=0.2 -> lower=0 upper=0 effort=0 velocity=0

Commit message: [Task 4.09] redone

File: rocr/urdf/rocr.urdf (robot description, URDF)
Before this commit: robot rocr, 9 links, 8 joints
Links:
- removed link dummy_link
Joints:
- removed joint dummy_joint

File: rocr/urdf/rocr_integration.urdf.xacro (robot description, xacro)
@@ -46,5 +46,5 @@
 	</gazebo>
 <!-- Add gazebo plugin for control here -->
-	<gazebo>
+	<!-- <gazebo>
 		<plugin name="gazebo_ros_control" filename="libgazebo_ros_control.so">
 			<robotNamespace>/rocr</robotNamespace>
@@ -52,5 +52,5 @@
 			<legacyModeNS>true</legacyModeNS>
 		</plugin>
-	</gazebo>
+	</gazebo> -->
 <!-- Create a joint between your robot and sensor -->
   <joint

Commit message: [Task 4.09] Modified model

File: rocr/urdf/rocr.urdf (robot description, URDF)
Before this commit: robot rocr, 8 links, 7 joints
Links:
- added link dummy_link
Joints:
- added joint dummy_joint: type fixed, parent dummy_link, child base_link
- joint joint_left_arm: limit lower=0 upper=0 effort=0 velocity=0 -> lower=-1.5 upper=3.5 effort=1 velocity=0.2
- joint joint_left_rim: axis 0 0 1 -> 0 0 -1
- joint joint_right_arm: limit lower=0 upper=0 effort=0 velocity=0 -> lower=-1.5 upper=3.5 effort=1 velocity=0.2

File: rocr/urdf/rocr_integration.urdf.xacro (robot description, xacro)
@@ -29,16 +29,16 @@
               	<range>
               		<min>0.10</min>
-              		<max>30.0</max>
-              		<resolution>0.01</resolution>
+              		<max>10.0</max>
+              		<resolution>0.1</resolution>
               	</range>
-              	<noise>
+              	<!-- <noise>
               		<type>gaussian</type>
               		<mean>0.0</mean>
               		<stddev>0.01</stddev>
-              	</noise>
+              	</noise> -->
             </ray>
             <plugin name="gazebo_ros_head_hokuyo_controller" filename="libgazebo_ros_laser.so">
             	<!-- Use topic name as /my_robot/scan -->
-				<topicName>/rocr/scan</topicName>
+				<topicName>/scan</topicName>
 				<frameName>laser_frame</frameName>
 			</plugin>
@@ -48,5 +48,5 @@
 	<!-- <gazebo>
 		<plugin name="gazebo_ros_control" filename="libgazebo_ros_control.so">
-			<robotNamespace>/rocr</robotNamespace>
+			<robotNamespace>/</robotNamespace>
 			<robotSimType>gazebo_ros_control/DefaultRobotHWSim</robotSimType>
 			<legacyModeNS>true</legacyModeNS>
