Commit message: [Task 4.05] Generated new file to check if URDF is okay

File: rocr/output.urdf (robot description, URDF)
Before this commit: robot rocr, 19 links, 18 joints
Links:
- removed link link_bolt
- removed link link_pinion
- link base_laser: geometry collision mesh filename=package://rocr/meshes/ydlidar.dae; visual mesh filename=package://rocr/meshes/ydlidar.dae
- link link_front_left_axle: mass 0.00966461047960184 -> 0.00980151610171137
- link link_front_left_rim: mass 0.0118944183288657 -> 0.0269891429421557
- link link_front_left_tyre: mass 0.000894793246519236 -> 0.00176187281891002
- link link_front_right_axle: mass 0.00966461047960182 -> 0.00980150843161576
- link link_front_right_rim: mass 0.0118944183288657 -> 0.0269891429421557
- link link_front_right_tyre: mass 0.000894793246519238 -> 0.00176187281891002
- link link_left_arm: mass 1.1924981757879 -> 0.160992890586137
- link link_rear_axle: mass 0.0146411571669772 -> 0.0152217234982576
- link link_rear_left_rim: mass 0.0118944183288657 -> 0.0269891429421556
- link link_rear_left_tyre: mass 0.000894793246519235 -> 0.00176187281891002
- link link_rear_right_rim: mass 0.0118944183288657 -> 0.0269891429421557
- link link_rear_right_tyre: mass 0.000894793246519237 -> 0.00176187281891002
- link link_right_arm: mass 1.22458311377959 -> 0.165316765586137
Joints:
- removed joint joint_bolt
- removed joint joint_pinion
- joint joint_front_left_axle: limit lower=-.35 upper=0.35 effort=1 velocity=0 -> lower=0 upper=0.0 effort=1 velocity=0; origin xyz=-0.16 -0.074 -0.0346 rpy=-1.5708 0 -1.5708 -> xyz=-0.16 -0.074 -0.0346 rpy=1.5708 0 -1.6484
- joint joint_front_left_rim: origin xyz=0.009 0.027 0 rpy=-1.5708 -0.51596 1.5708 -> xyz=0.0030721 -0.027 0 rpy=-1.5708 1.1039 1.5708
- joint joint_front_left_tyre: origin xyz=0 0 -0.006 rpy=0 0 0.53015 -> xyz=0 0 0 rpy=3.1416 0 -0.81007
- joint joint_front_right_axle: limit lower=-0.35 upper=0.35 effort=1 velocity=0 -> lower=0 upper=0 effort=1 velocity=0
- joint joint_front_right_rim: origin xyz=0.009 -0.027 0 rpy=1.5708 0.2483 -1.5708 -> xyz=0.003 -0.027 0 rpy=1.5708 -0.93241 -1.5708
- joint joint_front_right_tyre: origin xyz=0 0 -0.006 rpy=0 0 1.197 -> xyz=0 0 -0.012 rpy=0 0 0.63839
- joint joint_left_arm: axis 0 0 0 -> 0 0 1; limit lower=0 upper=0 effort=0 velocity=0 -> lower=-1.5 upper=3.5 effort=1 velocity=0.2; origin xyz=-0.214 -0.11955 -0.074 rpy=1.5708 0 0 -> xyz=-0.214 0.066422 -0.072 rpy=1.5708 0 0
- joint joint_rear_axle: origin xyz=-0.04 0 -0.0616 rpy=1.5707963267949 0.707024824141767 0 -> xyz=-0.04 0 -0.0616 rpy=1.5708 0 0
- joint joint_rear_left_rim: origin xyz=0 0 0.089 rpy=3.14159265358979 0 -0.351698544940136 -> xyz=0 0 0.089 rpy=3.1416 0 -2.7485
- joint joint_rear_left_tyre: origin xyz=0 0 0.00600000000000001 rpy=3.14159265358979 0 3.14159265358979 -> xyz=0 0 0.012 rpy=3.14159265358979 0 -2.74849784316327
- joint joint_rear_right_rim: origin xyz=0 0 0 rpy=0 0 0.24991380443404 -> xyz=0 0 0 rpy=0 0 0
- joint joint_rear_right_tyre: origin xyz=0 0 0 rpy=0 0 2.8695961764224 -> xyz=0 0 0 rpy=0 0 0
- joint joint_right_arm: axis 0 0 0 -> 0 0 1; limit lower=0 upper=0 effort=0 velocity=0 -> lower=-1.5 upper=3.5 effort=1 velocity=0.2; origin xyz=-0.36753 0.030166 -0.074 rpy=1.5708 0 0 -> xyz=-0.36753 0 -0.072 rpy=1.5708 0 0
- joint laser_chassis: origin xyz=-0.36 0 0.032 rpy=0 0 3.14 -> xyz=-0.25 -0.05 0.028 rpy=0 0 3.14
